File: hardware/ATT.kicad_sch (KiCad schematic)
At the start: 59 parts, among them J1 Conn_01x04, J2 Conn_01x04, J3 UART, J4 I2C1, J5 I2C2, J6 I2C3, J7 I2C4, J8 SERVO, J9 RPI, Q1 2N7000, Q2 2N7000, Q3 2N7000, Q4 2N7000, Q5 IRLZ44N, SW1 SW_DPST, SW2 ON/OFF, U1 Espressif_ESP32-S3-DevKitC1, U2 74HCT245N, U3 TB6600, U4 TB6600, U5 PC817

Commit message: Finalized-ish electronic hardware schematics
Parts:
- removed C1, C10, C3, C8, C9: 100nF, symbol Device:C
- removed C2, C4: 1uF, symbol Device:C_Polarized
- removed C5, C6, C7: 470uF, symbol Device:C_Polarized
- removed D1, D2, D3: R, symbol Device:LED
- removed D4: B, symbol Device:LED
- removed D5: 1N5819, Diode_THT:D_DO-41_SOD81_P10.16mm_Horizontal, symbol Diode:1N5819
- removed J1, J2: Conn_01x04, symbol Connector_Generic:Conn_01x04
- removed J3: UART, symbol Connector_Generic:Conn_01x06
- removed J4: I2C1, symbol Connector_Generic:Conn_01x04
- removed J5: I2C2, symbol Connector_Generic:Conn_01x04
- removed J6: I2C3, symbol Connector_Generic:Conn_01x04
- removed J7: I2C4, symbol Connector_Generic:Conn_01x04
- removed J8: SERVO, symbol Connector_Generic:Conn_01x03
- removed J9: RPI, symbol Connector_Generic:Conn_01x02
- removed Q1, Q2, Q3, Q4: 2N7000, Package_TO_SOT_THT:TO-92_Inline, symbol Transistor_FET:2N7000
- removed Q5: IRLZ44N, Package_TO_SOT_THT:TO-220-3_Vertical, symbol Transistor_FET:IRLZ44N
- removed R1, R2, R3: 4.7k, symbol Device:R
- removed R10, R12, R8: 100k, symbol Device:R
- removed R11, R13, R15, R17, R23, R9: 100, symbol Device:R
- removed R14, R16, R21: 10k, symbol Device:R
- removed R18: 1k, symbol Device:R
- removed R19, R20: 40m, symbol Device:R
- removed R22: 6.8k, symbol Device:R
- removed R4, R5, R6: 68, symbol Device:R
- removed R7: 33, symbol Device:R
- removed SW1: SW_DPST, symbol Switch:SW_DPST
- removed SW2: ON/OFF, symbol Switch:SW_Push
- removed U1: Espressif_ESP32-S3-DevKitC1, symbol MCU_Module_own:Espressif_ESP32-S3-DevKitC1
- removed U2: 74HCT245N, 74HCT245N:DIP254P762X420-20, symbol 74HCT245N:74HCT245N
- removed U3, U4: TB6600, symbol ATT:TB6600
- removed U5: PC817, Package_DIP:DIP-4_W7.62mm, symbol Isolator:PC817
Connections:
- no-connect marks 22 -> 0
Other:
- added sheet Controller (controller.kicad_sch)
- added sheet Power (power.kicad_sch)
- title: (none) -> ATT - Turret system schematic
